File: hardware_rp2040_minisdr/hardware_rp2040_minisdr.kicad_sch (KiCad schematic)
At the start: 0 parts

Commit message: started with schematic
Parts:
- added C1: C, symbol Device:C
- added C10, C11, C12, C13, C14, C15, C6, C7, C9: 100n, symbol Device:C
- added C16, C8: 1u, symbol Device:C
- added C2, C3: 15p, symbol Device:C
- added C4, C5: 10u, symbol Device:C
- added D1: ESDS314DBVR, SOT95P280X145-5N, symbol USER:ESDS314DBVR
- added J1: Conn_Coaxial_Small, symbol Connector:Conn_Coaxial_Small
- added J2: USB_A, symbol Connector:USB_A
- added R1: R, symbol Device:R
- added R2, R3: 27, symbol Device:R
- added R4: 1k, symbol Device:R
- added U1: RP2040, Package_DFN_QFN:QFN-56-1EP_7x7mm_P0.4mm_EP3.2x3.2mm, symbol MCU_RaspberryPi:RP2040
- added U2: W25Q128JVS, Package_SO:SOIC-8_5.3x5.3mm_P1.27mm, symbol Memory_Flash:W25Q128JVS
- added U3: AMS1117-3.3, Package_TO_SOT_SMD:SOT-223-3_TabPin2, symbol Regulator_Linear:AMS1117-3.3
- added Y1: Crystal_GND24, symbol Device:Crystal_GND24
Connections:
- new net: C2.1, R4.1, Y1.1
- new net: R4.2, U1.21 (XOUT)
- new net: C3.2, U1.20 (XIN), Y1.3
- new net: R3.2, U1.46 (USB_DM)
- new net: R2.1, U1.47 (USB_DP)
- new net: C4.1, J2.1 (VBUS), U3.3 (VI)
- new net 1v1: C6.1, C7.1, C8.1, U1.23 (DVDD), U1.45 (VREG_VOUT), U1.50 (DVDD)
- new net 3v3: C10.1, C11.1, C12.1, C13.1, C14.1, C15.1, C16.1, C5.1, C9.1, U1.1 (IOVDD), U1.10 (IOVDD), U1.22 (IOVDD), U1.26 (RUN), U1.33 (IOVDD), U1.42 (IOVDD), U1.43 (ADC_AVDD), U1.44 (VREG_IN), U1.48 (USB_VDD), U1.49 (IOVDD), U2.8 (VCC), U3.2 (VO)
- new net GND: C10.2, C11.2, C12.2, C13.2, C14.2, C15.2, C16.2, C2.2, C3.1, C4.2, C5.2, C6.2, C7.2, C8.2, C9.2, D1.2 (GND), J1.2 (Ext), J2.4 (GND), J2.5 (Shield), U1.19 (TESTEN), U1.57 (GND), U2.4 (GND), U3.1 (GND), Y1.2, Y1.4
- new net QSPI_SCLK: U1.52 (QSPI_SCLK), U2.6 (CLK)
- new net QSPI_SD0: U1.53 (QSPI_SD0), U2.5 (DI/IO_{0})
- new net QSPI_SD1: U1.55 (QSPI_SD1), U2.2 (DO/IO_{1})
- new net QSPI_SD2: U1.54 (QSPI_SD2), U2.3 (~{WP}/IO_{2})
- new net QSPI_SD3: U1.51 (QSPI_SD3), U2.7 (~{HOLD}/~{RESET}/IO_{3})
- new net QSPI_SS: U1.56 (QSPI_SS), U2.1 (~{CS})
- new net SWCLK: U1.24 (SWCLK)
- new net SWD: U1.25 (SWD)
- new net USB_DN: D1.5 (I/O4), J2.2 (D-), R3.1
- new net USB_DP: D1.4 (I/O3), J2.3 (D+), R2.2

Commit message: schematic
Parts:
- added C17, C18, C20, C21: 100n, symbol Device:C
- added C19, C22: 10u, symbol Device:C
- added IC1: PSA4-5043+, PSA45043, symbol RF:PSA4-5043+
- added IC2: ADE-11X+, SOTFL254P691X284-6N, symbol RF:ADE-11X+
- added IC3: SI5351A-B-GTR, SOP50P490X110-10N, symbol RF:SI5351A-B-GTR
- added IC4: GALI-84+, GALI5, symbol RF:GALI-84+
- added L1, L2: 220n, symbol Device:L
- added R5: 1k, symbol Device:R
- added R6: 50, symbol Device:R
- added SW1: SW_Push, symbol Switch:SW_Push
Connections:
- net GND: now also C19.1, IC1.2 (GND_1), IC1.4 (GND_2), IC2.1 (GROUND_1), IC2.4 (GROUND_2), IC2.5 (GROUND_3), IC4.2 (GROUND_1), IC4.4 (GROUND_2), SW1.1
- net QSPI_SS: now also R5.2
- net at J1.1 (In): now also C17.1
- net VBUS: now reaches C4.1, J2.1 (VBUS), U3.3 (VI)
- net VBUS: now also C19.2, C22.1, L1.1, R6.2
- new net: C21.1, IC2.6 (LO)
- new net: C21.2, IC4.3 (RF-OUT_&_DC-IN), L2.1
- new net: C18.1, IC1.1 (RF-OUT_&_DC-IN), L1.2
- new net: C17.2, IC1.3 (RF_IN)
- new net: C18.2, IC2.2 (RF)
- new net: R5.1, SW1.2
- new net: L2.2, R6.1
- new net: C20.2, IC4.1 (RF-IN)
Other:
- note added: "Connect this"
- moved on the sheet: J1

Commit message: schematic
Parts:
- added C23, C24: 22p, symbol Device:C
- added Y2: Crystal_GND24, symbol Device:Crystal_GND24
Connections:
- net 3v3: now also IC3.1 (VDD), IC3.7 (VDDO)
- net GND: now also C22.2, IC3.8 (GND), C23.1, C24.2, Y2.2, Y2.4
- net at IC3.10 (CLK0): now also C20.1
- net at IC3.2 (XA): now also C23.2, Y2.3
- net at IC3.3 (XB): now also C24.1, Y2.1
- net SCL: now reaches IC3.4 (SCL)
- net SDA: now reaches IC3.5 (SDA)
Other:
- note removed: "Connect this"

Commit message: schematic
Parts:
- added C25: 10n, symbol Device:C
- added C26: 100n, symbol Device:C
- added IC5: ADCS7476AIMFX_NOPB, SOT95P280X145-6N, symbol Analog_ADC:ADCS7476AIMFX_NOPB
- added L3, L4: 15u, symbol Device:L
Connections:
- net 3v3: now also IC5.1 (VDD)
- net GND: now also C25.2, IC5.2 (GND)
- net at IC2.3 (IF): now also L3.2
- new net: C25.1, L3.1, L4.2
- new net: C26.1, IC5.3 (VIN)
- new net: C26.2, L4.1
- new net ADC_CS: IC5.6 (~{CS})
- new net ADC_MISO: IC5.5 (SDATA)
- new net ADC_SCLK: IC5.4 (SCLK)

Commit message: schematic
Parts:
- removed C1: C, symbol Device:C
- removed R1: R, symbol Device:R
Changed lines of the file:
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@@
-	(symbol
-		(lib_id "Device:C")
-		(at 154.94 39.37 0)
-		(unit 1)
-		(exclude_from_sim no)
-		(in_bom yes)
-		(on_board yes)
-		(dnp no)
-		(fields_autoplaced yes)
-		(property "Reference" "C1"
-			(at 158.75 38.0999 0)
-			(effects
-				(font
-					(size 1.27 1.27)
-				)
-				(justify left)
-			)
-		)
-		(property "Value" "C"
-			(at 158.75 40.6399 0)
-			(effects
-				(font
-					(size 1.27 1.27)
-				)
-				(justify left)
-			)
-		)
-		(property "Footprint" ""
-			(at 155.9052 43.18 0)
-			(effects
-				(font
-					(size 1.27 1.27)
-				)
-				(hide yes)
-			)
-		)
-		(property "Datasheet" "~"
-			(at 154.94 39.37 0)
-			(effects
-				(font
-					(size 1.27 1.27)
-				)
-				(hide yes)
-			)
-		)
-		(property "Description" "Unpolarized capacitor"
-			(at 154.94 39.37 0)
-			(effects
-				(font
-					(size 1.27 1.27)
-				)
-				(hide yes)
-			)
-		)
-		(pin "2"
-		)
-		(pin "1"
-		)
-		(instances
-			(project ""
-				(path "/a9470e8c-e7c5-4ac0-a905-81d12777e86b"
-					(reference "C1")
-					(unit 1)
-				)
-			)
-		)
-	)
 	(symbol
 		(lib_id "Device:C")
@@
 					(unit 1)
 				)
-			)
-		)
-	)
-	(symbol
-		(lib_id "Device:R")
-		(at 156.21 27.94 0)
-		(unit 1)
-		(exclude_from_sim no)
-		(in_bom yes)
-		(on_board yes)
-		(dnp no)
-		(fields_autoplaced yes)
-		(property "Reference" "R1"
-			(at 158.75 26.6699 0)
-			(effects
-				(font
-					(size 1.27 1.27)
-				)
-				(justify left)
-			)
-		)
-		(property "Value" "R"
-			(at 158.75 29.2099 0)
-			(effects
-				(font
-					(size 1.27 1.27)
-				)
-				(justify left)
-			)
-		)
-		(property "Footprint" ""
-			(at 154.432 27.94 90)
-			(effects
-				(font
-					(size 1.27 1.27)
-				)
-				(hide yes)
-			)
-		)
-		(property "Datasheet" "~"
-			(at 156.21 27.94 0)
-			(effects
-				(font
-					(size 1.27 1.27)
-				)
-				(hide yes)
-			)
-		)
-		(property "Description" "Resistor"
-			(at 156.21 27.94 0)
-			(effects
-				(font
-					(size 1.27 1.27)
-				)
-				(hide yes)
-			)
-		)
-		(pin "2"
-		)
-		(pin "1"
-		)
-		(instances
-			(project ""
-				(path "/a9470e8c-e7c5-4ac0-a905-81d12777e86b"
-					(reference "R1")
-					(unit 1)
-				)

Commit message: board
Connections:
- net ADC_CS: now also U1.13 (GPIO10)
- net ADC_MISO: now also U1.12 (GPIO9)
- net ADC_SCLK: now also U1.14 (GPIO11)
- net SCL: now also U1.28 (GPIO17)
- net SDA: now also U1.27 (GPIO16)
Changed lines of the file:
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@@
+		)
+	)
+	(global_label "ADC_SCLK"
+		(shape input)
+		(at 228.6 96.52 0)
+		(fields_autoplaced yes)
+		(effects
+			(font
+				(size 1.27 1.27)
+			)
+			(justify left)
+		)
+		(property "Intersheetrefs" "${INTERSHEET_REFS}"
+			(at 240.959 96.52 0)
+			(effects
+				(font
+					(size 1.27 1.27)
+				)
+				(justify left)
+				(hide yes)
+			)
 		)
 	)
@@
 		)
 	)
+	(global_label "ADC_CS"
+		(shape input)
+		(at 228.6 93.98 0)
+		(fields_autoplaced yes)
+		(effects
+			(font
+				(size 1.27 1.27)
+			)
+			(justify left)
+		)
+		(property "Intersheetrefs" "${INTERSHEET_REFS}"
+			(at 238.6609 93.98 0)
+			(effects
+				(font
+					(size 1.27 1.27)
+				)
+				(justify left)
+				(hide yes)
+			)
+		)
+	)
+	(global_label "SCL"
+		(shape input)
+		(at 228.6 111.76 0)
+		(fields_autoplaced yes)
+		(effects
+			(font
+				(size 1.27 1.27)
+			)
+			(justify left)
+		)
+		(property "Intersheetrefs" "${INTERSHEET_REFS}"
+			(at 235.0928 111.76 0)
+			(effects
+				(font
+					(size 1.27 1.27)
+				)
+				(justify left)
+				(hide yes)
+			)
+		)
+	)
+	(global_label "ADC_MISO"
+		(shape input)
+		(at 228.6 91.44 0)
+		(fields_autoplaced yes)
+		(effects
+			(font
+				(size 1.27 1.27)
+			)
+			(justify left)
+		)
+		(property "Intersheetrefs" "${INTERSHEET_REFS}"
+			(at 240.7776 91.44 0)
+			(effects
+				(font
+					(size 1.27 1.27)
+				)
+				(justify left)
+				(hide yes)
+			)
+		)
+	)
 	(global_label "GND"
 		(shape input)
@@
 				(hide yes)
 			)
+		)
+	)
+	(global_label "SDA"
+		(shape input)
+		(at 228.6 109.22 0)
+		(fields_autoplaced yes)
+		(effects
+			(font
+				(size 1.27 1.27)
+			)
+			(justify left)
+		)
+		(property "Intersheetrefs" "${INTERSHEET_REFS}"
+			(at 235.1533 109.22 0)
+			(effects
+				(font
+					(size 1.27 1.27)
+				)
+				(justify left)
+				(hide yes)
+			)

Commit message: board
Parts:
- C10, C11, C12, C13, C14, C15, C17, C18, C2, C20, C21, C23, C24, C25, C26, C3, C6, C7, C9: footprint (none) -> Capacitor_SMD:C_0402_1005Metric
- D1: footprint SOT95P280X145-5N -> (none)
- IC1: footprint PSA45043 -> (none)
- IC2: footprint SOTFL254P691X284-6N -> (none)
- IC3: footprint SOP50P490X110-10N -> (none)
- IC4: footprint GALI5 -> (none)
- IC5: footprint SOT95P280X145-6N -> (none)
- J1: footprint (none) -> Connector_Coaxial:SMA_Amphenol_132289_EdgeMount
Changed lines of the file:
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@@
 			)
 		)
-		(property "Footprint" "SOP50P490X110-10N"
+		(property "Footprint" ""
 			(at 153.67 243.51 0)
 			(effects
@@
 			)
 		)
-		(property "Footprint" ""
+		(property "Footprint" "Connector_Coaxial:SMA_Amphenol_132289_EdgeMount"
 			(at 29.21 106.68 0)
 			(effects
@@
 			)
 		)
-		(property "Footprint" ""
+		(property "Footprint" "Capacitor_SMD:C_0402_1005Metric"
 			(at 247.3452 44.45 0)
 			(effects
@@
 			)
 		)
-		(property "Footprint" ""
+		(property "Footprint" "Capacitor_SMD:C_0402_1005Metric"
 			(at 77.1652 130.81 0)
 			(effects
@@
 			)
 		)
-		(property "Footprint" ""
+		(property "Footprint" "Capacitor_SMD:C_0402_1005Metric"
 			(at 224.4852 44.45 0)
 			(effects
@@
 			)
 		)
-		(property "Footprint" "PSA45043"
+		(property "Footprint" ""
 			(at 45.72 14.3 0)
 			(effects
@@
 			)
 		)
-		(property "Footprint" "SOT95P280X145-5N"
+		(property "Footprint" ""
 			(at 55.88 172.39 0)
 			(effects
@@
 			)
 		)
-		(property "Footprint" ""
+		(property "Footprint" "Capacitor_SMD:C_0402_1005Metric"
 			(at 155.9052 133.35 0)
 			(effects
@@
 			)
 		)
-		(property "Footprint" "SOTFL254P691X284-6N"
+		(property "Footprint" ""
 			(at 72.39 213.03 0)
 			(effects
@@
 			)
 		)
-		(property "Footprint" ""
+		(property "Footprint" "Capacitor_SMD:C_0402_1005Metric"
 			(at 39.37 133.6548 0)
 			(effects
@@
 			)
 		)
-		(property "Footprint" ""
+		(property "Footprint" "Capacitor_SMD:C_0402_1005Metric"
 			(at 254.9652 44.45 0)
 			(effects
@@
 			)
 		)
-		(property "Footprint" "SOT95P280X145-6N"
+		(property "Footprint" ""
 			(at 66.04 251.13 0)
 			(effects
@@
 			)
 		)
-		(property "Footprint" ""
+		(property "Footprint" "Capacitor_SMD:C_0402_1005Metric"
 			(at 239.7252 44.45 0)
 			(effects
@@
 			)
 		)
-		(property "Footprint" "GALI5"
+		(property "Footprint" ""
 			(at 91.44 32.08 0)
 			(effects
@@
 			)
 		)
-		(property "Footprint" ""
+		(property "Footprint" "Capacitor_SMD:C_0402_1005Metric"
 			(at 262.5852 44.45 0)
 			(effects
@@
 			)
 		)
-		(property "Footprint" ""
+		(property "Footprint" "Capacitor_SMD:C_0402_1005Metric"
 			(at 187.6552 48.26 0)
 			(effects
@@
 			)
 		)
-		(property "Footprint" ""
+		(property "Footprint" "Capacitor_SMD:C_0402_1005Metric"
 			(at 29.5148 147.32 0)
 			(effects
@@
 			)
 		)
-		(property "Footprint" ""
+		(property "Footprint" "Capacitor_SMD:C_0402_1005Metric"
 			(at 108.9152 162.56 0)
 			(effects
@@
 			)
 		)
-		(property "Footprint" ""
+		(property "Footprint" "Capacitor_SMD:C_0402_1005Metric"
 			(at 195.2752 48.26 0)
 			(effects
@@
 			)
 		)
-		(property "Footprint" ""
+		(property "Footprint" "Capacitor_SMD:C_0402_1005Metric"
 			(at 216.8652 44.45 0)
 			(effects
@@
 			)
 		)
-		(property "Footprint" ""
+		(property "Footprint" "Capacitor_SMD:C_0402_1005Metric"
 			(at 38.1 105.7148 0)
 			(effects
@@
 			)
 		)
-		(property "Footprint" ""
+		(property "Footprint" "Capacitor_SMD:C_0402_1005Metric"
 			(at 106.68 108.2548 0)
 			(effects
@@
 			)
 		)
-		(property "Footprint" ""
+		(property "Footprint" "Capacitor_SMD:C_0402_1005Metric"
 			(at 132.3848 127 0)
 			(effects
@@
 			)
 		)
-		(property "Footprint" ""
+		(property "Footprint" "Capacitor_SMD:C_0402_1005Metric"
 			(at 108.9152 147.32 0)
 			(effects
@@
 			)
 		)
-		(property "Footprint" ""
+		(property "Footprint" "Capacitor_SMD:C_0402_1005Metric"
 			(at 232.1052 44.45 0)
 			(effects
@@
 			)
 		)
-		(property "Footprint" ""
+		(property "Footprint" "Capacitor_SMD:C_0402_1005Metric"
 			(at 155.9052 114.3 0)
 			(effects

Commit message: board
Parts:
- C16, C8: footprint (none) -> Capacitor_SMD:C_0402_1005Metric
- C19, C22, C4, C5: footprint (none) -> Capacitor_SMD:C_0805_2012Metric
- D1: footprint (none) -> user_imported_devices:ESDS314BVR_SOT95P280X145-5N
- IC1: footprint (none) -> user_imported_devices:PSA45043
- IC2: footprint (none) -> user_imported_devices:ADE-11X+_SOTFL254P691X284-6N
- IC3: footprint (none) -> user_imported_devices:SI5351_SOP50P490X110-10N
- IC4: footprint (none) -> user_imported_devices:GALI5
- IC5: footprint (none) -> user_imported_devices:ADCS7476_SOT95P280X145-6N
- L1, L2, L3, L4: footprint (none) -> Inductor_SMD:L_0805_2012Metric
- R2, R3, R4, R5, R6: footprint (none) -> Resistor_SMD:R_0402_1005Metric
- SW1: footprint (none) -> Button_Switch_SMD:SW_SPST_PTS810
- Y1, Y2: footprint (none) -> Crystal:Crystal_SMD_3225-4Pin_3.2x2.5mm
Changed lines of the file:
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@@
 			)
 		)
-		(property "Footprint" ""
+		(property "Footprint" "user_imported_devices:SI5351_SOP50P490X110-10N"
 			(at 153.67 243.51 0)
 			(effects
@@
 			)
 		)
-		(property "Footprint" ""
+		(property "Footprint" "Resistor_SMD:R_0402_1005Metric"
 			(at 171.45 126.238 90)
 			(effects
@@
 			)
 		)
-		(property "Footprint" ""
+		(property "Footprint" "user_imported_devices:PSA45043"
 			(at 45.72 14.3 0)
 			(effects
@@
 			)
 		)
-		(property "Footprint" ""
+		(property "Footprint" "user_imported_devices:ESDS314BVR_SOT95P280X145-5N"
 			(at 55.88 172.39 0)
 			(effects
@@
 			)
 		)
-		(property "Footprint" ""
+		(property "Footprint" "Capacitor_SMD:C_0402_1005Metric"
 			(at 192.7352 57.15 0)
 			(effects
@@
 			)
 		)
-		(property "Footprint" ""
+		(property "Footprint" "user_imported_devices:ADE-11X+_SOTFL254P691X284-6N"
 			(at 72.39 213.03 0)
 			(effects
@@
 			)
 		)
-		(property "Footprint" ""
+		(property "Footprint" "Resistor_SMD:R_0402_1005Metric"
 			(at 123.952 81.28 90)
 			(effects
@@
 			)
 		)
-		(property "Footprint" ""
+		(property "Footprint" "Capacitor_SMD:C_0805_2012Metric"
 			(at 84.1248 96.52 0)
 			(effects
@@
 			)
 		)
-		(property "Footprint" ""
+		(property "Footprint" "Inductor_SMD:L_0805_2012Metric"
 			(at 83.82 130.81 0)
 			(effects
@@
 			)
 		)
-		(property "Footprint" ""
+		(property "Footprint" "Capacitor_SMD:C_0805_2012Metric"
 			(at 67.0052 53.34 0)
 			(effects
@@
 			)
 		)
-		(property "Footprint" ""
+		(property "Footprint" "Capacitor_SMD:C_0402_1005Metric"
 			(at 218.1352 57.15 0)
 			(effects
@@
 			)
 		)
-		(property "Footprint" ""
+		(property "Footprint" "user_imported_devices:ADCS7476_SOT95P280X145-6N"
 			(at 66.04 251.13 0)
 			(effects
@@
 			)
 		)
-		(property "Footprint" ""
+		(property "Footprint" "Resistor_SMD:R_0402_1005Metric"
 			(at 168.91 80.518 90)
 			(effects
@@
 			)
 		)
-		(property "Footprint" ""
+		(property "Footprint" "Button_Switch_SMD:SW_SPST_PTS810"
 			(at 120.65 72.39 0)
 			(effects
@@
 			)
 		)
-		(property "Footprint" ""
+		(property "Footprint" "user_imported_devices:GALI5"
 			(at 91.44 32.08 0)
 			(effects
@@
 			)
 		)
-		(property "Footprint" ""
+		(property "Footprint" "Resistor_SMD:R_0402_1005Metric"
 			(at 85.852 135.89 90)
 			(effects
@@
 			)
 		)
-		(property "Footprint" ""
+		(property "Footprint" "Crystal:Crystal_SMD_3225-4Pin_3.2x2.5mm"
 			(at 107.95 151.13 0)
 			(effects
@@
 			)
 		)
-		(property "Footprint" ""
+		(property "Footprint" "Capacitor_SMD:C_0805_2012Metric"
 			(at 92.4052 53.34 0)
 			(effects
@@
 			)
 		)
-		(property "Footprint" ""
+		(property "Footprint" "Crystal:Crystal_SMD_3225-4Pin_3.2x2.5mm"
 			(at 154.94 120.65 0)
 			(effects
@@
 			)
 		)
-		(property "Footprint" ""
+		(property "Footprint" "Capacitor_SMD:C_0805_2012Metric"
 			(at 80.01 140.6652 0)
 			(effects
@@
 			)
 		)
-		(property "Footprint" ""
+		(property "Footprint" "Inductor_SMD:L_0805_2012Metric"
 			(at 30.48 129.54 0)
 			(effects
@@
 			)
 		)
-		(property "Footprint" ""
+		(property "Footprint" "Inductor_SMD:L_0805_2012Metric"
 			(at 93.98 100.33 0)
 			(effects
@@
 			)
 		)
-		(property "Footprint" ""
+		(property "Footprint" "Inductor_SMD:L_0805_2012Metric"
 			(at 30.48 139.7 0)
 			(effects
@@
 			)
 		)
-		(property "Footprint" ""
+		(property "Footprint" "Resistor_SMD:R_0402_1005Metric"
 			(at 168.91 74.422 90)
 			(effects
