File: hardware_rp2040_minisdr/hardware_rp2040_minisdr.kicad_pcb (KiCad board)
At the start: 4 copper layers, 74.2 x 20 mm, 51 parts, among them IC1 PSA4-5043+, IC2 ADE-11X+, IC3 SI5351A-B-GTR, IC4 GALI-84+, IC5 ADCS7476AIMFX_NOPB, J1 Conn_Coaxial_Small, J2 USB_A, SW1 SW_Push, U1 RP2040, U2 W25Q128JVS, U3 AMS1117S-3.3, Y1 Crystal_GND24, Y2 Crystal_GND24

Commit message: silkscreen stuff
Routing:
- net GND: track 101.4 -> 124.8 mm
Other:
- board text added: "Made By Keyaan!"
- board text added: "RP2040-mini-SDR"
Changed lines of the file:
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@@
 		(layer "Edge.Cuts")
+	)
+	(gr_text "RP2040-mini-SDR\n"
+		(at 161.75 87.75 0)
+		(layer "F.SilkS")
+		(effects
+			(font
+				(size 1 1)
+				(thickness 0.1)
+			)
+			(justify left bottom)
+		)
+	)
+	(gr_text "Made By Keyaan!"
+		(at 200.75 93.25 0)
+		(layer "B.SilkS")
+		(effects
+			(font
+				(size 1 1)
+				(thickness 0.1)
+			)
+			(justify left bottom mirror)
+		)
 	)
 	(segment
@@
 		(net 1)
 	)
+	(segment
+		(start 211.75 99.1125)
+		(end 211.8875 99.25)
+		(width 0.2)
+		(layer "B.Cu")
+		(net 1)
+	)
+	(segment
+		(start 213.1375 92)
+		(end 211.8875 90.75)
+		(width 0.2)
+		(layer "B.Cu")
+		(net 1)
+	)
+	(segment
+		(start 210 92)
+		(end 210.6375 92)
+		(width 0.2)
+		(layer "B.Cu")
+		(net 1)
+	)
+	(segment
+		(start 211.75 99.3875)
+		(end 211.8875 99.25)
+		(width 0.2)
+		(layer "B.Cu")
+		(net 1)
+	)
+	(segment
+		(start 210 100.5)
+		(end 210.6375 100.5)
+		(width 0.2)
+		(layer "B.Cu")
+		(net 1)
+	)
+	(segment
+		(start 211.75 89.5)
+		(end 211.75 90.6125)
+		(width 0.2)
+		(layer "B.Cu")
+		(net 1)
+	)
+	(segment
+		(start 210.6375 98)
+		(end 211.8875 99.25)
+		(width 0.2)
+		(layer "B.Cu")
+		(net 1)
+	)
+	(segment
+		(start 212.25 99.25)
+		(end 211.8875 99.25)
+		(width 0.2)
+		(layer "B.Cu")
+		(net 1)
+	)
+	(segment
+		(start 210 98)
+		(end 210.6375 98)
+		(width 0.2)
+		(layer "B.Cu")
+		(net 1)
+	)
+	(segment
+		(start 213.1375 100.5)
+		(end 211.8875 99.25)
+		(width 0.2)
+		(layer "B.Cu")
+		(net 1)
+	)
+	(segment
+		(start 211.75 90.6125)
+		(end 211.8875 90.75)
+		(width 0.2)
+		(layer "B.Cu")
+		(net 1)
+	)
+	(segment
+		(start 211.75 100.5)
+		(end 211.75 99.3875)
+		(width 0.2)
+		(layer "B.Cu")
+		(net 1)
+	)
+	(segment
+		(start 213.5 92)
+		(end 213.1375 92)
+		(width 0.2)
+		(layer "B.Cu")
+		(net 1)
+	)
+	(segment
+		(start 210 89.5)
+		(end 210.6375 89.5)
+		(width 0.2)
+		(layer "B.Cu")
+		(net 1)
+	)
+	(segment
+		(start 213.5 100.5)
+		(end 213.1375 100.5)
+		(width 0.2)
+		(layer "B.Cu")
+		(net 1)
+	)
+	(segment
+		(start 211.75 92)
+		(end 211.75 90.8875)
+		(width 0.2)
+		(layer "B.Cu")
+		(net 1)
+	)
+	(segment
+		(start 213.1375 89.5)
+		(end 211.8875 90.75)
+		(width 0.2)
+		(layer "B.Cu")
+		(net 1)
+	)
+	(segment
+		(start 211.75 90.8875)
+		(end 211.8875 90.75)
+		(width 0.2)
+		(layer "B.Cu")
+		(net 1)
+	)
+	(segment
+		(start 213.5 98)
+		(end 212.25 99.25)
+		(width 0.2)
+		(layer "B.Cu")
+		(net 1)
+	)
+	(segment
+		(start 210.6375 100.5)
+		(end 211.8875 99.25)
+		(width 0.2)
+		(layer "B.Cu")
+		(net 1)
+	)
+	(segment
+		(start 210.6375 89.5)
+		(end 211.8875 90.75)
+		(width 0.2)
+		(layer "B.Cu")
+		(net 1)
+	)
+	(segment
+		(start 211.75 98)
+		(end 211.75 99.1125)
+		(width 0.2)
+		(layer "B.Cu")
+		(net 1)
+	)
+	(segment
+		(start 210.6375 92)
+		(end 211.8875 90.75)
+		(width 0.2)
+		(layer "B.Cu")
+		(net 1)
+	)
+	(segment
+		(start 213.5 89.5)
+		(end 213.1375 89.5)
+		(width 0.2)
+		(layer "B.Cu")
+		(net 1)
+	)

Commit message: idk
Other:
- board text added: "Made By Keyaan! For Hackclub Highway!"
- board text removed: "Made By Keyaan!"

Commit message: silkscreen designs
Parts:
- added G***: LOGO, LOGO, B.Cu at (194.6, 98.7)
- added REF**: ESD-Logo_8.9x8mm_SilkScreen, Symbol:ESD-Logo_8.9x8mm_SilkScreen, B.Cu at (158.2, 97.5)
Other:
- board text added: "https://github.com/Keyaan-07/rp2040-mini-SDR"

Commit message: added Do not touch in silkscreen
Other:
- board text added: "DO NOT TOUCH"
Changed lines of the file:
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@@
+		)
+	)
+	(gr_text "DO NOT TOUCH"
+		(at 163.977762 104 0)
+		(layer "B.SilkS")
+		(effects
+			(font
+				(size 1 1)
+				(thickness 0.1)
+			)
+			(justify left bottom mirror)
 		)
 	)
